File: pcb/neverx_daugther/neverx_daugther.kicad_sch (KiCad schematic)
At the start: 19 parts, among them J1 IN, J2 UL, J3 UR, J4 LL, J5 LR, Q1 BC807, U1 HX711

Commit message: Fixed wrongtraces
Connections:
- net GND: now also J1.5 (Pin_5)
- no-connect marks 4 -> 3
Changed lines of the file:
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@@
 		(at 92.71 49.53)
-	)
-	(no_connect
-		(at 105.41 49.53)
 	)
 	(wire
@@
 					(unit 1)
 				)
+			)
+		)
+	)
+	(symbol
+		(lib_id "power:GND")
+		(at 105.41 49.53 270)
+		(unit 1)
+		(exclude_from_sim no)
+		(in_bom yes)
+		(on_board yes)
+		(dnp no)
+		(property "Reference" "#PWR020"
+			(at 99.06 49.53 0)
+			(effects
+				(font
+					(size 1.27 1.27)
+				)
+				(hide yes)
+			)
+		)
+		(property "Value" "GND"
+			(at 100.33 49.53 90)
+			(effects
+				(font
+					(size 1.27 1.27)
+				)
+			)
+		)
+		(property "Footprint" ""
+			(at 105.41 49.53 0)
+			(effects
+				(font
+					(size 1.27 1.27)
+				)
+				(hide yes)
+			)
+		)
+		(property "Datasheet" ""
+			(at 105.41 49.53 0)
+			(effects
+				(font
+					(size 1.27 1.27)
+				)
+				(hide yes)
+			)
+		)
+		(property "Description" "Power symbol creates a global label with name \"GND\" , ground"
+			(at 105.41 49.53 0)
+			(effects
+				(font
+					(size 1.27 1.27)
+				)
+				(hide yes)
+			)
+		)
+		(pin "1"
+		)
+		(instances
+			(project "neverx_daugther"
+				(path "/e83e0b8f-abf0-4910-b5b8-3548662d20ae"
+					(reference "#PWR020")
+					(unit 1)
+				)
