File: pcb/neverx_main/neverx_main.kicad_pcb (KiCad board)
At the start: 2 copper layers, 80 x 125 mm, 18 parts, among them J1 DB1, J2 DB1, J3 DB1, J4 DB1, J5 DB1, J6 DB1, SW1 VAL, SW2 CONF, U1 LilyGO_T-SIM7080G-S3, U3 IPS_240_240

Commit message: Fixed wrongtraces
Connections:
- J1 pad 5: unconnected-(J1-Pin_5-Pad5) -> GND
